File: main_board/main_board.kicad_pcb (KiCad board)
At the start: 2 copper layers, 64 parts, among them J1 USB_B_Micro, J2 Conn_02x13_Odd_Even, J3 Conn_02x13_Odd_Even, Q1 DMP2170, Q2 DMP2170, U1 MIC5504-3.3YM5, U2 USBLC6-2SC6, U3 93LC56B, U4 FT2232H, Y1 12MHz

Commit message: Updates when doing some layout testing
Parts:
- added G***: LOGO, logos:crucible.kicad_14, F.Cu at (120.1, 80.9)
- added R17: 4.7K, Resistor_SMD:R_0603_1608Metric_Pad1.05x0.95mm_HandSolder, F.Cu at (144.1, 117.5)
- added R18: 4.7K, Resistor_SMD:R_0603_1608Metric_Pad1.05x0.95mm_HandSolder, F.Cu at (146.6, 116.7)
- added R19: 4.7K, Resistor_SMD:R_0603_1608Metric_Pad1.05x0.95mm_HandSolder, F.Cu at (146.5, 113.7)
- added R20: 4.7K, Resistor_SMD:R_0603_1608Metric_Pad1.05x0.95mm_HandSolder, F.Cu at (152.5, 112.0)
- moved C2 98.6 mm to (89.8, 103.7), turned to 90 degrees
- moved C1 92.6 mm to (87.5, 104.4), turned to 90 degrees
- moved C9 92.2 mm to (115.0, 109.4), turned to 90 degrees
- moved MK3 89.5 mm to (158.4, 75.0)
- moved C7 89.3 mm to (113.0, 98.5), turned to 270 degrees
- moved C4 88.9 mm to (102.6, 103.4), turned to 90 degrees
- moved C3 88.6 mm to (100.4, 102.9), turned to 90 degrees
- moved TP2 85.0 mm to (83.8, 105.9)
- moved U1 81.9 mm to (95.8, 105.4)
- moved C6 80.7 mm to (109.4, 99.0), turned to 270 degrees
- moved C8 72.0 mm to (112.3, 108.8), turned to 90 degrees
- moved C5 71.5 mm to (88.6, 114.0), turned to 0 degrees
- moved R2 70.6 mm to (91.5, 117.7)
- moved R5 69.8 mm to (91.0, 111.6), turned to 180 degrees
- moved C15 69.7 mm to (125.0, 101.1)
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Connections:
- net /USB_Bridge/VIO renamed VIO
- J2 pad 10: SDA -> SCL
- J2 pad 11: CFGOUT -> CFGRST
- J2 pad 12: CFGRST -> CFGOUT
- J2 pad 9: SCL -> SDA
Routing:
- net GND: track 0.00 -> 62.3 mm, vias 0 -> 30
- net BC7: track 0.00 -> 45.9 mm, vias 0 -> 2
- net RESET#: track 0.00 -> 45.6 mm, vias 0 -> 2
- net VPLL: track 0.00 -> 44.3 mm, vias 0 -> 2
- net BC5: track 0.00 -> 44.0 mm, vias 0 -> 2
- net BC6: track 0.00 -> 43.8 mm, vias 0 -> 2
- net AD1: track 0.00 -> 43.3 mm
- net BC4: track 0.00 -> 41.7 mm, vias 0 -> 2
- net AD2: track 0.00 -> 41.0 mm
- net VIO: track 0.00 -> 38.0 mm
- net CFGOUT: track 0.00 -> 38.0 mm, vias 0 -> 1
- net VPHY: track 0.00 -> 37.3 mm, vias 0 -> 2
- net SCL: track 0.00 -> 37.2 mm, vias 0 -> 2
- net AC1: track 0.00 -> 36.8 mm
- net SDA: track 0.00 -> 36.3 mm, vias 0 -> 2
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- added copper zone on B.Cu, net GND
- added copper zone on F.Cu, net Net-(J1-Pad6)
- added copper zone on F.Cu, net VBUS
- added copper zone on F.Cu, net VCC3V3
Other:
- board outline added: 93.8 x 63.4 mm
- net class Default: clearance 0.2 -> 0.15; trace_width 0.25 -> 0.15; via_dia 0.8 -> 0.6; via_drill 0.4 -> 0.35
- net class USB added: clearance 0.15, trace_width 0.15, via_dia 0.6, via_drill 0.35
- rule trace_clearance: 0.2 -> 0.15
- rule trace_min: 0.2 -> 0.15
- rule via_min_drill: 0.3 -> 0.35
- rule via_min_size: 0.4 -> 0.6
- board text added: "Achenarian Empire Imperial Debugger Mk. 1"
