File: sub-modules/rs485_module/rs485_module/rs485_module.kicad_sch (KiCad schematic)
At the start: 14 parts, among them J1 Conn_02x06_Odd_Even, J2 TX_EN_Sel, J3 TX Pol, J4 RX Pol, J5 TERM_EN, J6 RS422/485, J9 MKDS 1/ 5-3,5, U1 74LVC1GU04DRL, U2 ADM3491ExR

Commit message: Sorting out BOMs
Signed-off-by: Marc Kelly <mpkelly@achenar.co.uk>
Parts:
- C1: value 100n -> 100nF; MFN (none) -> Generic X7R; MFP (none) -> 100nF; SUPPLIER (none) -> Mouser; SUPPLIER_PN (none) -> 581-06035C104JAT2A62
- J1: MFN (none) -> Wurth; MFP (none) -> 613012243121; SUPPLIER (none) -> Mouser; SUPPLIER_PN (none) -> 710-613012243121
- J2: MFN (none) -> Samtec; MFP (none) -> FTS-103-04-F-D; SUPPLIER (none) -> Mouser; SUPPLIER_PN (none) -> 200-FTS-103-04-F-D
- J3, J4, J6: MFN (none) -> Wurth; MFP (none) -> 62200421121; SUPPLIER (none) -> Mouser; SUPPLIER_PN (none) -> 710-62200421121
- J5: MFN (none) -> Harwin; MFP (none) -> M50-3530242; SUPPLIER (none) -> Mouser; SUPPLIER_PN (none) -> 855-M50-3530242
- J9: SUPPLIER (none) -> Mouser; SUPPLIER_PN (none) -> 651-1751277
- R1, R2, R4: value 10k -> 4.7k; MFN (none) -> Generic; MFP (none) -> 4.7k 1%; SUPPLIER (none) -> Mouser; SUPPLIER_PN (none) -> 594-MCT06030C4701FP5
- R3: MFN (none) -> Generic 1/4 W; MFP (none) -> 120R 1%; SUPPLIER (none) -> Mouser; SUPPLIER_PN (none) -> 279-CRGP0603F120R
- U1: MFN (none) -> Texas Instruments; MFP (none) -> SN74LVC1GU04DRLR; SUPPLIER (none) -> Mouser; SUPPLIER_PN (none) -> 595-SN74LVC1GU04DRLR
- U2: MFN (none) -> Renesas; MFP (none) -> ISL83076EIBZA; SUPPLIER (none) -> Mouser; SUPPLIER_PN (none) -> 968-ISL83076EIBZA
