File: sub-modules/rs485_module/rs485_module/rs485_module.kicad_sch (KiCad schematic)
At the start: 14 parts, among them J1 Conn_02x06_Odd_Even, J2 TX_EN_Sel, J3 TX Pol, J4 RX Pol, J5 TERM_EN, J6 RS422/485, J9 MKDS 1/ 5-3,5, U1 74LVC1GU04DRL, U2 ADM3491ExR

Commit message: Adding some Alt suppliers for suppler pns
Signed-off-by: Marc Kelly <mpkelly@achenar.co.uk>
Parts:
- C1: ALT_SUPPLIER (none) -> DigiKey; ALT_SUPPLIER_PN (none) -> 1276-1001-1-ND
- J1: ALT_SUPPLIER (none) -> DigiKey; ALT_SUPPLIER_PN (none) -> 732-613012243121-ND
- J2: ALT_SUPPLIER (none) -> DigiKey; ALT_SUPPLIER_PN (none) -> FTS-103-04-F-D-ND
- J3, J4, J6: ALT_SUPPLIER (none) -> DigiKey; ALT_SUPPLIER_PN (none) -> 732-5372-ND
- J5: ALT_SUPPLIER (none) -> DigiKey; ALT_SUPPLIER_PN (none) -> 952-3598-ND
- J9: ALT_SUPPLIER (none) -> DigiKey; ALT_SUPPLIER_PN (none) -> 277-5827-ND
- R1, R2, R4: ALT_SUPPLIER (none) -> DigiKey; ALT_SUPPLIER_PN (none) -> RC0402FR-074K7L
- R3: ALT_SUPPLIER (none) -> DigiKey; ALT_SUPPLIER_PN (none) -> CMP0603QFX-1200ELF
- U1: ALT_SUPPLIER (none) -> DigiKey; ALT_SUPPLIER_PN (none) -> 296-18657-1-ND
- U2: ALT_SUPPLIER (none) -> DigiKey; ALT_SUPPLIER_PN (none) -> ISL83076EIBZA-ND
Changed lines of the file:
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@@
 			)
 		)
-		(property "ALT_SUPPLIER" ""
+		(property "ALT_SUPPLIER" "DigiKey"
 			(at 48.26 127 0)
 			(hide yes)
@@
 			)
 		)
-		(property "ALT_SUPPLIER_PN" ""
+		(property "ALT_SUPPLIER_PN" "FTS-103-04-F-D-ND"
 			(at 48.26 127 0)
 			(hide yes)
@@
 			)
 		)
+		(property "ALT_SUPPLIER" "DigiKey"
+			(at 160.02 83.82 0)
+			(hide yes)
+			(show_name no)
+			(do_not_autoplace no)
+			(effects
+				(font
+					(size 1.27 1.27)
+				)
+			)
+		)
+		(property "ALT_SUPPLIER_PN" "ISL83076EIBZA-ND"
+			(at 160.02 83.82 0)
+			(hide yes)
+			(show_name no)
+			(do_not_autoplace no)
+			(effects
+				(font
+					(size 1.27 1.27)
+				)
+			)
+		)
 		(pin "5"
 		)
@@
 			)
 		)
+		(property "ALT_SUPPLIER" "DigiKey"
+			(at 90.17 134.62 0)
+			(hide yes)
+			(show_name no)
+			(do_not_autoplace no)
+			(effects
+				(font
+					(size 1.27 1.27)
+				)
+			)
+		)
+		(property "ALT_SUPPLIER_PN" "RC0402FR-074K7L"
+			(at 90.17 134.62 0)
+			(hide yes)
+			(show_name no)
+			(do_not_autoplace no)
+			(effects
+				(font
+					(size 1.27 1.27)
+				)
+			)
+		)
 		(pin "2"
 		)
@@
 			)
 		)
+		(property "ALT_SUPPLIER" "DigiKey"
+			(at 55.88 119.38 0)
+			(hide yes)
+			(show_name no)
+			(do_not_autoplace no)
+			(effects
+				(font
+					(size 1.27 1.27)
+				)
+			)
+		)
+		(property "ALT_SUPPLIER_PN" "RC0402FR-074K7L"
+			(at 55.88 119.38 0)
+			(hide yes)
+			(show_name no)
+			(do_not_autoplace no)
+			(effects
+				(font
+					(size 1.27 1.27)
+				)
+			)
+		)
 		(pin "2"
 		)
@@
 			)
 		)
-		(property "ALT_SUPPLIER" ""
+		(property "ALT_SUPPLIER" "DigiKey"
 			(at 194.31 63.5 0)
 			(hide yes)
@@
 			)
 		)
-		(property "ALT_SUPPLIER_PN" ""
+		(property "ALT_SUPPLIER_PN" "952-3598-ND"
 			(at 194.31 63.5 0)
 			(hide yes)
@@
 			)
 		)
+		(property "ALT_SUPPLIER" "DigiKey"
+			(at 87.63 113.03 0)
+			(hide yes)
+			(show_name no)
+			(do_not_autoplace no)
+			(effects
+				(font
+					(size 1.27 1.27)
+				)
+			)
+		)
+		(property "ALT_SUPPLIER_PN" "732-5372-ND"
+			(at 87.63 113.03 0)
+			(hide yes)
+			(show_name no)
+			(do_not_autoplace no)
+			(effects
+				(font
+					(size 1.27 1.27)
+				)
+			)
+		)
 		(pin "2"
 		)
@@
 			)
 		)
-		(property "ALT_SUPPLIER" ""
+		(property "ALT_SUPPLIER" "DigiKey"
 			(at 251.46 85.09 0)
 			(hide yes)
@@
 			)
 		)
-		(property "ALT_SUPPLIER_PN" ""
+		(property "ALT_SUPPLIER_PN" "277-5827-ND"
 			(at 251.46 85.09 0)
 			(hide yes)
@@
 		)
 		(property "SUPPLIER_PN" "595-SN74LVC1GU04DRLR"
+			(at 49.53 149.86 0)
+			(hide yes)
+			(show_name no)
+			(do_not_autoplace no)
+			(effects
+				(font
+					(size 1.27 1.27)
+				)
+			)
+		)
+		(property "ALT_SUPPLIER" "DigiKey"
+			(at 49.53 149.86 0)
+			(hide yes)
+			(show_name no)
+			(do_not_autoplace no)
+			(effects
+				(font
+					(size 1.27 1.27)
+				)
+			)
+		)
+		(property "ALT_SUPPLIER_PN" "296-18657-1-ND"
 			(at 49.53 149.86 0)
 			(hide yes)
@@
 			)
 		)
+		(property "ALT_SUPPLIER" "DigiKey"
+			(at 146.05 64.77 0)
+			(hide yes)
+			(show_name no)
+			(do_not_autoplace no)
+			(effects
+				(font
+					(size 1.27 1.27)
+				)
+			)
+		)
+		(property "ALT_SUPPLIER_PN" "1276-1001-1-ND"
+			(at 146.05 64.77 0)
+			(hide yes)
+			(show_name no)
+			(do_not_autoplace no)
+			(effects
+				(font
+					(size 1.27 1.27)
+				)
+			)
+		)
 		(pin "2"
 		)
@@
 			)
 		)
+		(property "ALT_SUPPLIER" "DigiKey"
+			(at 82.55 139.7 0)
+			(hide yes)
+			(show_name no)
+			(do_not_autoplace no)
+			(effects
+				(font
+					(size 1.27 1.27)
+				)
+			)
+		)
+		(property "ALT_SUPPLIER_PN" "732-5372-ND"
+			(at 82.55 139.7 0)
+			(hide yes)
+			(show_name no)
+			(do_not_autoplace no)
+			(effects
+				(font
+					(size 1.27 1.27)
+				)
+			)
+		)
 		(pin "2"
 		)
@@
 		)
 		(property "SUPPLIER_PN" "279-CRGP0603F120R"
+			(at 190.5 71.12 90)
+			(hide yes)
+			(show_name no)
+			(do_not_autoplace no)
+			(effects
+				(font
+					(size 1.27 1.27)
+				)
+			)
+		)
+		(property "ALT_SUPPLIER" "DigiKey"
+			(at 190.5 71.12 90)
+			(hide yes)
+			(show_name no)
+			(do_not_autoplace no)
+			(effects
+				(font
+					(size 1.27 1.27)
+				)
+			)
+		)
+		(property "ALT_SUPPLIER_PN" "CMP0603QFX-1200ELF"
 			(at 190.5 71.12 90)
 			(hide yes)
@@
 			)
 		)
-		(property "ALT_SUPPLIER" ""
+		(property "ALT_SUPPLIER" "DigiKey"
 			(at 55.88 81.28 0)
 			(hide yes)
@@
 			)
 		)
-		(property "ALT_SUPPLIER_PN" ""
+		(property "ALT_SUPPLIER_PN" "732-613012243121-ND"
 			(at 55.88 81.28 0)
 			(hide yes)
@@
 		)
 		(property "SUPPLIER_PN" "710-62200421121"
+			(at 196.85 97.79 0)
+			(hide yes)
+			(show_name no)
+			(do_not_autoplace no)
+			(effects
+				(font
+					(size 1.27 1.27)
+				)
+			)
+		)
+		(property "ALT_SUPPLIER" "DigiKey"
+			(at 196.85 97.79 0)
+			(hide yes)
+			(show_name no)
+			(do_not_autoplace no)
+			(effects
+				(font
+					(size 1.27 1.27)
+				)
+			)
+		)
+		(property "ALT_SUPPLIER_PN" "732-5372-ND"
 			(at 196.85 97.79 0)
 			(hide yes)
@@
 			(at 95.25 118.11 0)
 			(hide yes)
+			(show_name no)
+			(do_not_autoplace no)
+			(effects
+				(font
+					(size 1.27 1.27)
+				)
+			)
+		)
+		(property "ALT_SUPPLIER" "DigiKey"
+			(at 95.25 118.11 0)
+			(hide yes)
+			(show_name no)
+			(do_not_autoplace no)
+			(effects
+				(font
+					(size 1.27 1.27)
+				)
+			)
+		)
+		(property "ALT_SUPPLIER_PN" "RC0402FR-074K7L"
+			(at 95.25 118.11 0)
+			(hide yes)
