File: sub-modules/rs232_module/rs232_module/rs232_module.kicad_sch (KiCad schematic)
At the start: 12 parts, among them J1 Conn_02x06_Odd_Even, J9 MPT 0,5/ 6-2,54, U1 ADM3312EARUZ-REEL7

Commit message: Adding some Alt suppliers for suppler pns
Signed-off-by: Marc Kelly <mpkelly@achenar.co.uk>
Parts:
- C1, C2, C3, C5, C6, C7: ALT_SUPPLIER (none) -> DigiKey; ALT_SUPPLIER_PN (none) -> 399-C0603C104J4RACTUCT-ND
- C8: ALT_SUPPLIER (none) -> DigiKey; ALT_SUPPLIER_PN (none) -> 399-10203-1-ND
- J1: ALT_SUPPLIER (none) -> DigiKey; ALT_SUPPLIER_PN (none) -> 732-613012243121-ND
- J9: ALT_SUPPLIER (none) -> DigiKey; ALT_SUPPLIER_PN (none) -> 277-1277-ND
- R1, R2: ALT_SUPPLIER (none) -> DigiKey; ALT_SUPPLIER_PN (none) -> RC0402FR-074K7L
- U1: ALT_SUPPLIER (none) -> DigiKey; ALT_SUPPLIER_PN (none) -> 505-ADM3312EARUZ-REEL7CT-ND
Changed lines of the file:
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@@
+			)
+		)
+		(property "ALT_SUPPLIER" "DigiKey"
+			(at 73.66 168.91 0)
+			(hide yes)
+			(show_name no)
+			(do_not_autoplace no)
+			(effects
+				(font
+					(size 1.27 1.27)
+				)
+			)
+		)
+		(property "ALT_SUPPLIER_PN" "RC0402FR-074K7L"
+			(at 73.66 168.91 0)
+			(hide yes)
+			(show_name no)
+			(do_not_autoplace no)
+			(effects
+				(font
+					(size 1.27 1.27)
+				)
 			)
 		)
@@
 			)
 		)
+		(property "ALT_SUPPLIER" "DigiKey"
+			(at 123.19 123.19 0)
+			(hide yes)
+			(show_name no)
+			(do_not_autoplace no)
+			(effects
+				(font
+					(size 1.27 1.27)
+				)
+			)
+		)
+		(property "ALT_SUPPLIER_PN" "399-C0603C104J4RACTUCT-ND"
+			(at 123.19 123.19 0)
+			(hide yes)
+			(show_name no)
+			(do_not_autoplace no)
+			(effects
+				(font
+					(size 1.27 1.27)
+				)
+			)
+		)
 		(pin "1"
 		)
@@
 		)
 		(property "SUPPLIER_PN" "581-06035C104JAT2A62"
+			(at 71.12 152.4 0)
+			(hide yes)
+			(show_name no)
+			(do_not_autoplace no)
+			(effects
+				(font
+					(size 1.27 1.27)
+				)
+			)
+		)
+		(property "ALT_SUPPLIER" "DigiKey"
+			(at 71.12 152.4 0)
+			(hide yes)
+			(show_name no)
+			(do_not_autoplace no)
+			(effects
+				(font
+					(size 1.27 1.27)
+				)
+			)
+		)
+		(property "ALT_SUPPLIER_PN" "399-C0603C104J4RACTUCT-ND"
 			(at 71.12 152.4 0)
 			(hide yes)
@@
 			)
 		)
+		(property "ALT_SUPPLIER" "DigiKey"
+			(at 64.77 163.83 0)
+			(hide yes)
+			(show_name no)
+			(do_not_autoplace no)
+			(effects
+				(font
+					(size 1.27 1.27)
+				)
+			)
+		)
+		(property "ALT_SUPPLIER_PN" "RC0402FR-074K7L"
+			(at 64.77 163.83 0)
+			(hide yes)
+			(show_name no)
+			(do_not_autoplace no)
+			(effects
+				(font
+					(size 1.27 1.27)
+				)
+			)
+		)
 		(pin "1"
 		)
@@
 			)
 		)
+		(property "ALT_SUPPLIER" "DigiKey"
+			(at 119.38 153.67 0)
+			(hide yes)
+			(show_name no)
+			(do_not_autoplace no)
+			(effects
+				(font
+					(size 1.27 1.27)
+				)
+			)
+		)
+		(property "ALT_SUPPLIER_PN" "399-C0603C104J4RACTUCT-ND"
+			(at 119.38 153.67 0)
+			(hide yes)
+			(show_name no)
+			(do_not_autoplace no)
+			(effects
+				(font
+					(size 1.27 1.27)
+				)
+			)
+		)
 		(pin "1"
 		)
@@
 			)
 		)
+		(property "ALT_SUPPLIER" "DigiKey"
+			(at 130.81 118.11 0)
+			(hide yes)
+			(show_name no)
+			(do_not_autoplace no)
+			(effects
+				(font
+					(size 1.27 1.27)
+				)
+			)
+		)
+		(property "ALT_SUPPLIER_PN" "399-C0603C104J4RACTUCT-ND"
+			(at 130.81 118.11 0)
+			(hide yes)
+			(show_name no)
+			(do_not_autoplace no)
+			(effects
+				(font
+					(size 1.27 1.27)
+				)
+			)
+		)
 		(pin "1"
 		)
@@
 			)
 		)
-		(property "ALT_SUPPLIER" ""
+		(property "ALT_SUPPLIER" "DigiKey"
 			(at 139.7 118.11 0)
 			(hide yes)
@@
 			)
 		)
-		(property "ALT_SUPPLIER_PN" ""
+		(property "ALT_SUPPLIER_PN" "399-10203-1-ND"
 			(at 139.7 118.11 0)
 			(hide yes)
@@
 			)
 		)
-		(property "ALT_SUPPLIER" ""
+		(property "ALT_SUPPLIER" "DigiKey"
 			(at 243.84 76.2 0)
 			(hide yes)
@@
 			)
 		)
-		(property "ALT_SUPPLIER_PN" ""
+		(property "ALT_SUPPLIER_PN" "277-1277-ND"
 			(at 243.84 76.2 0)
 			(hide yes)
@@
 			)
 		)
+		(property "ALT_SUPPLIER" "DigiKey"
+			(at 119.38 147.32 0)
+			(hide yes)
+			(show_name no)
+			(do_not_autoplace no)
+			(effects
+				(font
+					(size 1.27 1.27)
+				)
+			)
+		)
+		(property "ALT_SUPPLIER_PN" "399-C0603C104J4RACTUCT-ND"
+			(at 119.38 147.32 0)
+			(hide yes)
+			(show_name no)
+			(do_not_autoplace no)
+			(effects
+				(font
+					(size 1.27 1.27)
+				)
+			)
+		)
 		(pin "1"
 		)
@@
 			)
 		)
+		(property "ALT_SUPPLIER" "DigiKey"
+			(at 119.38 168.91 0)
+			(hide yes)
+			(show_name no)
+			(do_not_autoplace no)
+			(effects
+				(font
+					(size 1.27 1.27)
+				)
+			)
+		)
+		(property "ALT_SUPPLIER_PN" "399-C0603C104J4RACTUCT-ND"
+			(at 119.38 168.91 0)
+			(hide yes)
+			(show_name no)
+			(do_not_autoplace no)
+			(effects
+				(font
+					(size 1.27 1.27)
+				)
+			)
+		)
 		(pin "1"
 		)
@@
 			)
 		)
-		(property "ALT_SUPPLIER" ""
+		(property "ALT_SUPPLIER" "DigiKey"
 			(at 55.88 81.28 0)
 			(hide yes)
@@
 			)
 		)
-		(property "ALT_SUPPLIER_PN" ""
+		(property "ALT_SUPPLIER_PN" "732-613012243121-ND"
 			(at 55.88 81.28 0)
 			(hide yes)
@@
 			(at 95.25 148.59 0)
 			(hide yes)
+			(show_name no)
+			(do_not_autoplace no)
+			(effects
+				(font
+					(size 1.27 1.27)
+				)
+			)
+		)
+		(property "ALT_SUPPLIER" "DigiKey"
+			(at 95.25 148.59 0)
+			(hide yes)
+			(show_name no)
+			(do_not_autoplace no)
+			(effects
+				(font
+					(size 1.27 1.27)
+				)
+			)
+		)
+		(property "ALT_SUPPLIER_PN" "505-ADM3312EARUZ-REEL7CT-ND"
+			(at 95.25 148.59 0)
+			(hide yes)
