File: sub-modules/ttl_module/ttl_module/ttl_module.kicad_sch (KiCad schematic)
At the start: 14 parts, among them J1 Input, J2 Output, J3 VCC Selection, U1 SN74LVC2T45DCTR, U2 SN74LVC2T45DCTR, U3 SN74LVC1T45DCK

Commit message: Adding some Alt suppliers for suppler pns
Signed-off-by: Marc Kelly <mpkelly@achenar.co.uk>
Parts:
- C1, C2, C3, C4, C5, C6: ALT_SUPPLIER (none) -> DigiKey; ALT_SUPPLIER_PN (none) -> CL05B104KO5NNNC
- J1: ALT_SUPPLIER (none) -> DigiKey; ALT_SUPPLIER_PN (none) -> 732-613012243121-ND
- J2: ALT_SUPPLIER (none) -> DigiKey; ALT_SUPPLIER_PN (none) -> 952-3300-ND
- J3: ALT_SUPPLIER (none) -> DigiKey; ALT_SUPPLIER_PN (none) -> 952-3276-ND
- R1, R2: ALT_SUPPLIER (none) -> DigiKey; ALT_SUPPLIER_PN (none) -> CRCW06034K70FKEA
- U1, U2: ALT_SUPPLIER (none) -> DigiKey; ALT_SUPPLIER_PN (none) -> 296-16845-1-ND
- U3: ALT_SUPPLIER (none) -> DigiKey; ALT_SUPPLIER_PN (none) -> 296-16844-1-ND
Changed lines of the file:
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@@
 			)
 		)
-		(property "ALT_SUPPLIER" ""
+		(property "ALT_SUPPLIER" "DigiKey"
 			(at 55.88 137.16 0)
 			(hide yes)
@@
 			)
 		)
-		(property "ALT_SUPPLIER_PN" ""
+		(property "ALT_SUPPLIER_PN" "952-3276-ND"
 			(at 55.88 137.16 0)
 			(hide yes)
@@
 			)
 		)
-		(property "ALT_SUPPLIER" ""
+		(property "ALT_SUPPLIER" "DigiKey"
 			(at 135.89 152.4 0)
 			(hide yes)
@@
 			)
 		)
-		(property "ALT_SUPPLIER_PN" ""
+		(property "ALT_SUPPLIER_PN" "296-16844-1-ND"
 			(at 135.89 152.4 0)
 			(hide yes)
@@
 			)
 		)
+		(property "ALT_SUPPLIER" "DigiKey"
+			(at 130.81 138.43 90)
+			(hide yes)
+			(show_name no)
+			(do_not_autoplace no)
+			(effects
+				(font
+					(size 1.27 1.27)
+				)
+			)
+		)
+		(property "ALT_SUPPLIER_PN" "CL05B104KO5NNNC"
+			(at 130.81 138.43 90)
+			(hide yes)
+			(show_name no)
+			(do_not_autoplace no)
+			(effects
+				(font
+					(size 1.27 1.27)
+				)
+			)
+		)
 		(pin "1"
 		)
@@
 		)
 		(property "SUPPLIER_PN" "581-06035C104JAT2A62"
+			(at 140.97 87.63 90)
+			(hide yes)
+			(show_name no)
+			(do_not_autoplace no)
+			(effects
+				(font
+					(size 1.27 1.27)
+				)
+			)
+		)
+		(property "ALT_SUPPLIER" "DigiKey"
+			(at 140.97 87.63 90)
+			(hide yes)
+			(show_name no)
+			(do_not_autoplace no)
+			(effects
+				(font
+					(size 1.27 1.27)
+				)
+			)
+		)
+		(property "ALT_SUPPLIER_PN" "CL05B104KO5NNNC"
 			(at 140.97 87.63 90)
 			(hide yes)
@@
 			)
 		)
+		(property "ALT_SUPPLIER" "DigiKey"
+			(at 140.97 138.43 90)
+			(hide yes)
+			(show_name no)
+			(do_not_autoplace no)
+			(effects
+				(font
+					(size 1.27 1.27)
+				)
+			)
+		)
+		(property "ALT_SUPPLIER_PN" "CL05B104KO5NNNC"
+			(at 140.97 138.43 90)
+			(hide yes)
+			(show_name no)
+			(do_not_autoplace no)
+			(effects
+				(font
+					(size 1.27 1.27)
+				)
+			)
+		)
 		(pin "1"
 		)
@@
 			)
 		)
-		(property "ALT_SUPPLIER" ""
+		(property "ALT_SUPPLIER" "DigiKey"
 			(at 135.89 46.99 0)
 			(hide yes)
@@
 			)
 		)
-		(property "ALT_SUPPLIER_PN" ""
+		(property "ALT_SUPPLIER_PN" "296-16845-1-ND"
 			(at 135.89 46.99 0)
 			(hide yes)
@@
 			)
 		)
+		(property "ALT_SUPPLIER" "DigiKey"
+			(at 130.81 30.48 90)
+			(hide yes)
+			(show_name no)
+			(do_not_autoplace no)
+			(effects
+				(font
+					(size 1.27 1.27)
+				)
+			)
+		)
+		(property "ALT_SUPPLIER_PN" "CL05B104KO5NNNC"
+			(at 130.81 30.48 90)
+			(hide yes)
+			(show_name no)
+			(do_not_autoplace no)
+			(effects
+				(font
+					(size 1.27 1.27)
+				)
+			)
+		)
 		(pin "1"
 		)
@@
 		)
 		(property "SUPPLIER_PN" "581-06035C104JAT2A62"
+			(at 130.81 87.63 90)
+			(hide yes)
+			(show_name no)
+			(do_not_autoplace no)
+			(effects
+				(font
+					(size 1.27 1.27)
+				)
+			)
+		)
+		(property "ALT_SUPPLIER" "DigiKey"
+			(at 130.81 87.63 90)
+			(hide yes)
+			(show_name no)
+			(do_not_autoplace no)
+			(effects
+				(font
+					(size 1.27 1.27)
+				)
+			)
+		)
+		(property "ALT_SUPPLIER_PN" "CL05B104KO5NNNC"
 			(at 130.81 87.63 90)
 			(hide yes)
@@
 			)
 		)
+		(property "ALT_SUPPLIER" "DigiKey"
+			(at 140.97 30.48 90)
+			(hide yes)
+			(show_name no)
+			(do_not_autoplace no)
+			(effects
+				(font
+					(size 1.27 1.27)
+				)
+			)
+		)
+		(property "ALT_SUPPLIER_PN" "CL05B104KO5NNNC"
+			(at 140.97 30.48 90)
+			(hide yes)
+			(show_name no)
+			(do_not_autoplace no)
+			(effects
+				(font
+					(size 1.27 1.27)
+				)
+			)
+		)
 		(pin "1"
 		)
@@
 			)
 		)
+		(property "ALT_SUPPLIER" "DigiKey"
+			(at 113.03 106.68 90)
+			(hide yes)
+			(show_name no)
+			(do_not_autoplace no)
+			(effects
+				(font
+					(size 1.27 1.27)
+				)
+			)
+		)
+		(property "ALT_SUPPLIER_PN" "CRCW06034K70FKEA"
+			(at 113.03 106.68 90)
+			(hide yes)
+			(show_name no)
+			(do_not_autoplace no)
+			(effects
+				(font
+					(size 1.27 1.27)
+				)
+			)
+		)
 		(pin "2"
 		)
@@
 			)
 		)
+		(property "ALT_SUPPLIER" "DigiKey"
+			(at 113.03 152.4 90)
+			(hide yes)
+			(show_name no)
+			(do_not_autoplace no)
+			(effects
+				(font
+					(size 1.27 1.27)
+				)
+			)
+		)
+		(property "ALT_SUPPLIER_PN" "CRCW06034K70FKEA"
+			(at 113.03 152.4 90)
+			(hide yes)
+			(show_name no)
+			(do_not_autoplace no)
+			(effects
+				(font
+					(size 1.27 1.27)
+				)
+			)
+		)
 		(pin "2"
 		)
@@
 			)
 		)
-		(property "ALT_SUPPLIER" ""
+		(property "ALT_SUPPLIER" "DigiKey"
 			(at 233.68 83.82 0)
 			(hide yes)
@@
 			)
 		)
-		(property "ALT_SUPPLIER_PN" ""
+		(property "ALT_SUPPLIER_PN" "952-3300-ND"
 			(at 233.68 83.82 0)
 			(hide yes)
@@
 			)
 		)
-		(property "ALT_SUPPLIER" ""
+		(property "ALT_SUPPLIER" "DigiKey"
 			(at 135.89 104.14 0)
 			(hide yes)
@@
 			)
 		)
-		(property "ALT_SUPPLIER_PN" ""
+		(property "ALT_SUPPLIER_PN" "296-16845-1-ND"
 			(at 135.89 104.14 0)
 			(hide yes)
@@
 			)
 		)
-		(property "ALT_SUPPLIER" ""
+		(property "ALT_SUPPLIER" "DigiKey"
 			(at 55.88 81.28 0)
 			(hide yes)
@@
 			)
 		)
-		(property "ALT_SUPPLIER_PN" ""
+		(property "ALT_SUPPLIER_PN" "732-613012243121-ND"
 			(at 55.88 81.28 0)
 			(hide yes)
