File: USB_and_power.kicad_sch (KiCad schematic)
At the start: 48 parts, among them J5 USB_C_Receptacle_USB2.0_14P, SW1 ResetButton, U3 LM2594M-3.3, U4 FT4232H, U5 93LC54B, Y1 ABLS7M2-12.000MHZ-D2Y-T

Commit message: Update oscillator caps
Replaced with correct 27pf in schematic

Signed-off-by: Marc Kelly <mpkelly@achenar.co.uk>
Parts:
- C18, C19: value 100nF -> 27pf
Changed lines of the file:
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@@
 			)
 		)
-		(property "Value" "100nF"
+		(property "Value" "27pf"
 			(at 215.9 226.695 0)
 			(show_name no)
@@
 			)
 		)
-		(property "Value" "100nF"
+		(property "Value" "27pf"
 			(at 228.6 226.695 0)
 			(show_name no)
