File: USB_and_power.kicad_sch (KiCad schematic)
At the start: 48 parts, among them J5 USB_C_Receptacle_USB2.0_14P, SW1 ResetButton, U3 LM2594M-3.3, U4 FT4232H, U5 93LC54B, Y1 ABLS7M2-12.000MHZ-D2Y-T

Commit message: Update Alt suppliers for UK/EU ones
Signed-off-by: Marc Kelly <mpkelly@achenar.co.uk>
Parts:
- C1, C11, C13, C15, C17, C2, C20, C3, C4, C5, C6, C7: ALT_SUPPLIER DigiKey -> TME; ALT_SUPPLIER_PN 399-C0603C104J4RACTUCT-ND -> GRM188R71C104KA01D
- C10, C12: ALT_SUPPLIER DigiKey -> TME; ALT_SUPPLIER_PN 490-7203-1-ND -> LMK107BJ475KA-T
- C14: ALT_SUPPLIER DigiKey -> TME; ALT_SUPPLIER_PN 399-C0603C103J3RACAUTOCT-ND -> GRT1885C1E103FA02D
- C16: ALT_SUPPLIER DigiKey -> TME; ALT_SUPPLIER_PN 478-4949-1-ND -> CL10A335KP8NNNC
- C18, C19: ALT_SUPPLIER DigiKey -> TME; ALT_SUPPLIER_PN 399-C0603C104J4RACTUCT-ND -> CC0603JRNPO9270
- C8: ALT_SUPPLIER DigiKey -> TME; ALT_SUPPLIER_PN 478-3069-1-ND -> TAJB686K010R
- C9: ALT_SUPPLIER DigiKey -> TME; ALT_SUPPLIER_PN 10-EEE-FN1A151LCT-ND -> EEEFN1C151UP
- D19: ALT_SUPPLIER DigiKey -> TME; ALT_SUPPLIER_PN 1N5819HW-FDICT-ND -> SS1040-R1
- D20, D23: ALT_SUPPLIER DigiKey -> TME; ALT_SUPPLIER_PN ESD5Z2.5T1GOSCT-ND -> ESD7351XV2T1G
- D21: ALT_SUPPLIER DigiKey -> TME; ALT_SUPPLIER_PN 732-155060GS75300CT-ND -> KP-1608SGD
- D22: ALT_SUPPLIER DigiKey -> TME; ALT_SUPPLIER_PN 732-12014-1-ND -> RF-OUB191TS-CE
- F1: ALT_SUPPLIER DigiKey -> TME; ALT_SUPPLIER_PN 5923-0ZCJ0075AF2ECT-ND -> 0ZCJ0075AF2E
- J5: ALT_SUPPLIER DigiKey -> Farnell; ALT_SUPPLIER_PN 2223-UJ20-C-H-G-SMT-2A-P16-TRCT-ND -> 4839404
- L1, L2, L4: ALT_SUPPLIER DigiKey -> Farnell; ALT_SUPPLIER_PN 445-175372-1-ND -> 4065960
- L3: ALT_SUPPLIER DigiKey -> TME; ALT_SUPPLIER_PN SRN6045-101MCT-ND -> DJNR6045-101-S
- R17, R18: ALT_SUPPLIER DigiKey -> TME; ALT_SUPPLIER_PN RMCF0603FT10R0 -> HP03-10R1%
- R19, R24: ALT_SUPPLIER DigiKey -> TME; ALT_SUPPLIER_PN RC0603FR-0710KL -> HP03-10K1%
- R20: ALT_SUPPLIER DigiKey -> TME; ALT_SUPPLIER_PN RC0402FR-0712KL -> ERA3AEB123V
- R21, R28: ALT_SUPPLIER DigiKey -> TME; ALT_SUPPLIER_PN CAS06F0000CT -> MCT06030Z0000ZP500
- R22, R23: ALT_SUPPLIER DigiKey -> TME; ALT_SUPPLIER_PN RC0603FR-075K1L -> AR0603-5K1-0.1%
- R25: ALT_SUPPLIER DigiKey -> TME; ALT_SUPPLIER_PN YAG3590CT-ND -> ERA3AEB202V
- R26, R27: ALT_SUPPLIER DigiKey -> TME; ALT_SUPPLIER_PN RC0603FR-07330RL -> ARG0603-330R-0.5%
- SW1: ALT_SUPPLIER DigiKey -> TME; ALT_SUPPLIER_PN 2073-SWT0110-020016SSACT-ND -> SWT0110-020016SSA
- U3: ALT_SUPPLIER DigiKey -> TME; ALT_SUPPLIER_PN LM2594M-3.3/NOPB-ND -> LM2594M-3.3/NOPB
- U4: ALT_SUPPLIER (none) -> TME; ALT_SUPPLIER_PN (none) -> FT4232HL
- U5: value 93LC54B -> 93LC54A; ALT_SUPPLIER DigiKey -> TME; ALT_SUPPLIER_PN 93LC56B-I/MS-ND -> 93LC56A-I/SN; SUPPLIER_PN 579-93LC56B-I/MS -> 579-93LC56A-I/MS
- Y1: ALT_SUPPLIER DigiKey -> Farnell; ALT_SUPPLIER_PN 541-XT9MNLANA14M31818-ND -> 2467681
