File: imperial_debugger.kicad_sch (KiCad schematic)
At the start: 10 parts

Commit message: Adding some Alt suppliers for suppler pns
Signed-off-by: Marc Kelly <mpkelly@achenar.co.uk>
Parts:
- TP1, TP2: ALT_SUPPLIER (none) -> DigiKey; ALT_SUPPLIER_PN (none) -> 36-5006-ND
Changed lines of the file:
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@@
 			)
 		)
-		(property "ALT_SUPPLIER" ""
+		(property "ALT_SUPPLIER" "DigiKey"
 			(at 38.1 114.3 0)
 			(hide yes)
@@
 			)
 		)
-		(property "ALT_SUPPLIER_PN" ""
+		(property "ALT_SUPPLIER_PN" "36-5006-ND"
 			(at 38.1 114.3 0)
 			(hide yes)
@@
 			)
 		)
-		(property "ALT_SUPPLIER" ""
+		(property "ALT_SUPPLIER" "DigiKey"
 			(at 58.42 114.3 0)
 			(hide yes)
@@
 			)
 		)
-		(property "ALT_SUPPLIER_PN" ""
+		(property "ALT_SUPPLIER_PN" "36-5006-ND"
 			(at 58.42 114.3 0)
 			(hide yes)

Commit message: Update Alt suppliers for UK/EU ones
Signed-off-by: Marc Kelly <mpkelly@achenar.co.uk>
Parts:
- TP1, TP2: ALT_SUPPLIER DigiKey -> Farnell; ALT_SUPPLIER_PN 36-5006-ND -> 2301284
Changed lines of the file:
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@@
 			)
 		)
-		(property "ALT_SUPPLIER" "DigiKey"
+		(property "ALT_SUPPLIER" "Farnell"
 			(at 38.1 114.3 0)
 			(hide yes)
@@
 			)
 		)
-		(property "ALT_SUPPLIER_PN" "36-5006-ND"
+		(property "ALT_SUPPLIER_PN" "2301284"
 			(at 38.1 114.3 0)
 			(hide yes)
@@
 			)
 		)
-		(property "ALT_SUPPLIER" "DigiKey"
+		(property "ALT_SUPPLIER" "Farnell"
 			(at 58.42 114.3 0)
 			(hide yes)
@@
 			)
 		)
-		(property "ALT_SUPPLIER_PN" "36-5006-ND"
+		(property "ALT_SUPPLIER_PN" "2301284"
 			(at 58.42 114.3 0)
 			(hide yes)
