File: transceiver.kicad_sch (KiCad schematic)
At the start: 45 parts, among them J1 Conn_02x06_Odd_Even, J2 Conn_02x06_Odd_Even, J3 Conn_02x06_Odd_Even, J4 Conn_02x06_Odd_Even, Q1 FDV301N, Q2 FDV301N, U1 TLV75525PDBV, U2 TLV75518PDBV

Commit message: Adding some Alt suppliers for suppler pns
Signed-off-by: Marc Kelly <mpkelly@achenar.co.uk>
Parts:
- D1, D2, D24, D25, D3, D4, D5, D6: ALT_SUPPLIER (none) -> DigiKey; ALT_SUPPLIER_PN (none) -> 296-ESDS304DBVRCT-ND
- D10, D11, D12, D13, D14, D15, D16, D17, D18, D7, D8, D9: ALT_SUPPLIER (none) -> DigiKey; ALT_SUPPLIER_PN (none) -> 732-155060GS75300CT-ND
- J1, J2, J3, J4: ALT_SUPPLIER (none) -> DigiKey; ALT_SUPPLIER_PN (none) -> 10129382-912003BLF-ND
- JP1: ALT_SUPPLIER (none) -> DigiKey; ALT_SUPPLIER_PN (none) -> S9012E-04-ND
- Q1, Q2: ALT_SUPPLIER (none) -> DigiKey; ALT_SUPPLIER_PN (none) -> FDV301NCT-ND
- R1, R10, R11, R12, R13, R14, R2, R3, R4, R5, R6, R7, R8, R9: ALT_SUPPLIER (none) -> DigiKey; ALT_SUPPLIER_PN (none) -> RC0603FR-07330RL
- R15, R16: ALT_SUPPLIER (none) -> DigiKey; ALT_SUPPLIER_PN (none) -> RC0402FR-074K7L
- U1: ALT_SUPPLIER (none) -> DigiKey; ALT_SUPPLIER_PN (none) -> 296-51795-1-ND
- U2: ALT_SUPPLIER (none) -> DigiKey; ALT_SUPPLIER_PN (none) -> 296-50410-1-ND

Commit message: Update Alt suppliers for UK/EU ones
Signed-off-by: Marc Kelly <mpkelly@achenar.co.uk>
Parts:
- D1, D2, D24, D25, D3, D4, D5, D6: ALT_SUPPLIER DigiKey -> TME; ALT_SUPPLIER_PN 296-ESDS304DBVRCT-ND -> SP0504BAHTG-LF
- D10, D7, D8, D9: ALT_SUPPLIER DigiKey -> TME; ALT_SUPPLIER_PN 732-155060GS75300CT-ND -> KPH-1608YD
- D11, D12, D13, D14, D15, D16, D17, D18: ALT_SUPPLIER DigiKey -> TME; ALT_SUPPLIER_PN 732-155060GS75300CT-ND -> KP-1608SGD
- J1, J2, J3, J4: ALT_SUPPLIER DigiKey -> Farnell; ALT_SUPPLIER_PN 10129382-912003BLF-ND -> 3497357
- JP1: ALT_SUPPLIER DigiKey -> TME; ALT_SUPPLIER_PN S9012E-04-ND -> ZL322-2X4P
- Q1, Q2: ALT_SUPPLIER DigiKey -> TME; ALT_SUPPLIER_PN FDV301NCT-ND -> 2N7002-TP
- R1, R10, R11, R12, R13, R14, R2, R3, R4, R5, R6, R7, R8, R9: ALT_SUPPLIER DigiKey -> TME; ALT_SUPPLIER_PN RC0603FR-07330RL -> ARG0603-330R-0.5%
- R15, R16: ALT_SUPPLIER DigiKey -> TME; ALT_SUPPLIER_PN RC0402FR-074K7L -> HP03-4K71%
- U1: ALT_SUPPLIER DigiKey -> TME; ALT_SUPPLIER_PN 296-51795-1-ND -> AP2112K-2.5TRG1
- U2: ALT_SUPPLIER DigiKey -> TME; ALT_SUPPLIER_PN 296-50410-1-ND -> AP2112K-1.8TRG1
